File: clap.kicad_pcb (KiCad board)
At the start: 2 copper layers, 34 parts, among them J1 Screw_Terminal_01x01, J2 Screw_Terminal_01x01, J3 Screw_Terminal_01x01, J4 Screw_Terminal_01x01, K1 G5Q-1, Q1 BC337, Q2 BC337, U1 LM358, U2 CD4017BE, U3 NE555

Commit message: refactoring
Routing:
- net Net-(RV1-Pad1): track 8.07 -> 20.1 mm, vias 0 -> 1
- net /Vcc: track 101.8 -> 113.9 mm
Changed lines of the file:
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@@
-(kicad_pcb (version 20171130) (host pcbnew "(5.0.2)-1")
+(kicad_pcb (version 20171130) (host pcbnew "(5.1.5)-3")
   (general
     (thickness 1.6)
     (drawings 0)
-    (tracks 160)
+    (tracks 170)
     (zones 0)
     (modules 34)
@@
     (zone_45_only no)
     (trace_min 0.2)
-    (segment_width 0.2)
-    (edge_width 0.15)
     (via_size 0.8)
     (via_drill 0.4)
@@
     (uvia_min_size 0.2)
     (uvia_min_drill 0.1)
+    (edge_width 0.15)
+    (segment_width 0.2)
     (pcb_text_width 0.3)
     (pcb_text_size 1.5 1.5)
@@
   (segment (start 177.375 114.2) (end 177.475 114.1) (width 0.6) (layer F.Cu) (net 1))
   (segment (start 174.76 114.2) (end 177.375 114.2) (width 0.6) (layer F.Cu) (net 1))
+  (segment (start 168.075 105.725) (end 169.425 105.725) (width 0.6) (layer B.Cu) (net 1))
+  (segment (start 174.76 111.06) (end 174.76 114.2) (width 0.6) (layer B.Cu) (net 1))
+  (segment (start 169.425 105.725) (end 174.76 111.06) (width 0.6) (layer B.Cu) (net 1))
   (via (at 135.5 99.9) (size 0.8) (drill 0.4) (layers F.Cu B.Cu) (net 2))
   (segment (start 134.6 100.8) (end 135.5 99.9) (width 0.6) (layer F.Cu) (net 2))
@@
   (segment (start 141.675 115.025) (end 142.73 113.97) (width 0.6) (layer F.Cu) (net 20))
   (segment (start 126 110.8) (end 123.9 108.7) (width 0.6) (layer F.Cu) (net 21))
+  (segment (start 126.4 110.8) (end 126.4 110.8) (width 0.6) (layer F.Cu) (net 21))
+  (segment (start 123.9 108.7) (end 119.2 108.7) (width 0.6) (layer F.Cu) (net 21))
   (segment (start 126.4 110.8) (end 126 110.8) (width 0.6) (layer F.Cu) (net 21))
-  (segment (start 123.9 108.7) (end 119.2 108.7) (width 0.6) (layer F.Cu) (net 21))
+  (via (at 126.4 110.8) (size 0.8) (drill 0.4) (layers F.Cu B.Cu) (net 21))
+  (segment (start 126.8 110.8) (end 129.7 113.7) (width 0.6) (layer B.Cu) (net 21))
+  (segment (start 126.4 110.8) (end 126.8 110.8) (width 0.6) (layer B.Cu) (net 21))
+  (segment (start 132.22 118.42) (end 134.02 118.42) (width 0.6) (layer B.Cu) (net 21))
+  (segment (start 129.7 115.9) (end 132.22 118.42) (width 0.6) (layer B.Cu) (net 21))
+  (segment (start 129.7 113.7) (end 129.7 115.9) (width 0.6) (layer B.Cu) (net 21))
   (segment (start 174.36 116.74) (end 174.76 116.74) (width 0.6) (layer F.Cu) (net 27))
   (segment (start 172.96 118.14) (end 174.36 116.74) (width 0.6) (layer F.Cu) (net 27))
